File: ir_bisector_board/pcb_&_schematic/ir_bisector/ir_bisector.kicad_sch (KiCad schematic)
At the start: 14 parts, among them J1 01x03_Pin, J2 01x03_Pin, U1 TCRT1010, U2 TCRT1010, U3 TCRT1010, U4 AO3401

Commit message: sensor board finished
Parts:
- removed J2: 01x03_Pin, symbol Connector:Conn_01x03_Pin
- removed R7: 10k, symbol Device:R
- removed U4: AO3401, AO3401:SOT23, symbol AO3401:AO3401
- added J2: 01x02_Pin, Connector_PinHeader_1.00mm:PinHeader_1x02_P1.00mm_Vertical, symbol Connector:Conn_01x02_Pin
- C1: footprint (none) -> Capacitor_SMD:C_0603_1608Metric
- J1: footprint (none) -> Connector_PinHeader_1.00mm:PinHeader_1x03_P1.00mm_Vertical
- R1, R2, R3, R4, R5, R6: footprint (none) -> Resistor_SMD:R_0603_1608Metric
- U1, U2, U3: footprint TCRT1010_VIS -> TCRT1010:TCRT1010_VIS
Connections:
- net +3.3V_SUB is gone; now on net +3.3V: R1.2, R2.1, R3.2, R4.1, R5.2, R6.1
- net +3.3V: now also J2.1 (Pin_1)
- net GND: now also J2.2 (Pin_2)
